File: cnc_shield.sch (EAGLE design)
At the start: 14 parts, among them X4 1751248

Commit message: botoes de entrada
Parts:
- added S1, S2, S3: (no value), RepRapjr:10-XX-RPAD
Connections:
- new net N$16: S3.S, U$1.A0
- new net N$17: S1.S, U$1.A1
- new net N$18: S2.S, U$1.A2
- net GND: now also S1.P, S2.P, S3.P
Changed lines of the file:
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@@
 <part name="SUPPLY6" library="supply2" deviceset="VCC" device=""/>
 <part name="X4" library="con-phoenix-350" deviceset="1751248" device=""/>
+<part name="S1" library="RepRapjr" deviceset="10-XX-RPAD" device=""/>
+<part name="S2" library="RepRapjr" deviceset="10-XX-RPAD" device=""/>
+<part name="S3" library="RepRapjr" deviceset="10-XX-RPAD" device=""/>
+<part name="GND4" library="supply1" deviceset="GND" device=""/>
 </parts>
 <sheets>
@@
 <instance part="X4" gate="-1" x="97.79" y="148.59" rot="R180"/>
 <instance part="X4" gate="-2" x="97.79" y="156.21" rot="R180"/>
+<instance part="S1" gate="1" x="34.29" y="77.47" rot="R270"/>
+<instance part="S2" gate="1" x="34.29" y="66.04" rot="R270"/>
+<instance part="S3" gate="1" x="34.29" y="87.63" rot="R270"/>
+<instance part="GND4" gate="1" x="24.13" y="58.42"/>
 </instances>
 <busses>
@@
 <pinref part="GND3" gate="1" pin="GND"/>
 <wire x1="214.63" y1="129.54" x2="208.28" y2="129.54" width="0.1524" layer="91"/>
+</segment>
+<segment>
+<pinref part="S3" gate="1" pin="P"/>
+<pinref part="GND4" gate="1" pin="GND"/>
+<wire x1="29.21" y1="87.63" x2="24.13" y2="87.63" width="0.1524" layer="91"/>
+<wire x1="24.13" y1="87.63" x2="24.13" y2="77.47" width="0.1524" layer="91"/>
+<pinref part="S1" gate="1" pin="P"/>
+<wire x1="24.13" y1="77.47" x2="24.13" y2="66.04" width="0.1524" layer="91"/>
+<wire x1="24.13" y1="66.04" x2="24.13" y2="60.96" width="0.1524" layer="91"/>
+<wire x1="29.21" y1="77.47" x2="24.13" y2="77.47" width="0.1524" layer="91"/>
+<junction x="24.13" y="77.47"/>
+<pinref part="S2" gate="1" pin="P"/>
+<wire x1="29.21" y1="66.04" x2="24.13" y2="66.04" width="0.1524" layer="91"/>
+<junction x="24.13" y="66.04"/>
 </segment>
 </net>
@@
 </segment>
 </net>
+<net name="N$16" class="0">
+<segment>
+<pinref part="U$1" gate="G$1" pin="A0"/>
+<wire x1="63.5" y1="95.25" x2="43.18" y2="95.25" width="0.1524" layer="91"/>
+<wire x1="43.18" y1="95.25" x2="43.18" y2="87.63" width="0.1524" layer="91"/>
+<pinref part="S3" gate="1" pin="S"/>
+<wire x1="43.18" y1="87.63" x2="39.37" y2="87.63" width="0.1524" layer="91"/>
+</segment>
+</net>
+<net name="N$17" class="0">
+<segment>
+<pinref part="S1" gate="1" pin="S"/>
+<wire x1="39.37" y1="77.47" x2="45.72" y2="77.47" width="0.1524" layer="91"/>
+<wire x1="45.72" y1="77.47" x2="45.72" y2="92.71" width="0.1524" layer="91"/>
+<pinref part="U$1" gate="G$1" pin="A1"/>
+<wire x1="45.72" y1="92.71" x2="63.5" y2="92.71" width="0.1524" layer="91"/>
+</segment>
+</net>
+<net name="N$18" class="0">
+<segment>
+<pinref part="S2" gate="1" pin="S"/>
+<wire x1="39.37" y1="66.04" x2="48.26" y2="66.04" width="0.1524" layer="91"/>
+<wire x1="48.26" y1="66.04" x2="48.26" y2="90.17" width="0.1524" layer="91"/>
+<pinref part="U$1" gate="G$1" pin="A2"/>
+<wire x1="48.26" y1="90.17" x2="63.5" y2="90.17" width="0.1524" layer="91"/>
+</segment>
+</net>

Commit message: alimentaçao
Connections:
- net GND: now also U$1.GND
- net VCC: now also U$1.5.5V
Changed lines of the file:
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@@
 <part name="S3" library="RepRapjr" deviceset="10-XX-RPAD" device=""/>
 <part name="GND4" library="supply1" deviceset="GND" device=""/>
+<part name="SUPPLY7" library="supply2" deviceset="VCC" device=""/>
+<part name="GND5" library="supply1" deviceset="GND" device=""/>
 </parts>
 <sheets>
@@
 <instance part="S3" gate="1" x="34.29" y="87.63" rot="R270"/>
 <instance part="GND4" gate="1" x="24.13" y="58.42"/>
+<instance part="SUPPLY7" gate="G$1" x="58.42" y="78.74"/>
+<instance part="GND5" gate="1" x="58.42" y="66.04"/>
 </instances>
 <busses>
@@
 <wire x1="151.13" y1="144.78" x2="153.67" y2="144.78" width="0.1524" layer="91"/>
 </segment>
+<segment>
+<pinref part="SUPPLY7" gate="G$1" pin="VCC"/>
+<wire x1="58.42" y1="76.2" x2="58.42" y2="74.93" width="0.1524" layer="91"/>
+<pinref part="U$1" gate="G$1" pin="5.5V"/>
+<wire x1="58.42" y1="74.93" x2="63.5" y2="74.93" width="0.1524" layer="91"/>
+</segment>
 </net>
 <net name="GND" class="0">
@@
 <junction x="24.13" y="66.04"/>
 </segment>
+<segment>
+<pinref part="GND5" gate="1" pin="GND"/>
+<wire x1="58.42" y1="68.58" x2="58.42" y2="69.85" width="0.1524" layer="91"/>
+<pinref part="U$1" gate="G$1" pin="GND"/>
+<wire x1="58.42" y1="69.85" x2="63.5" y2="69.85" width="0.1524" layer="91"/>
+</segment>
 </net>

Commit message: 1 versao board
Connections:
- removed net GND_MOT: C1.-, C2.-, C3.-, U$2.GND@0, U$3.GND@0, U$4.GND@0, X4-2.K
- net GND: now also C1.-, C2.-, C3.-, U$2.GND@0, U$3.GND@0, U$4.GND@0, X4-2.K
Changed lines of the file:
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@@
 <wire x1="58.42" y1="69.85" x2="63.5" y2="69.85" width="0.1524" layer="91"/>
 </segment>
-</net>
-<net name="GND_MOT" class="0">
 <segment>
-<pinref part="U$4" gate="G$1" pin="GND@0"/>
-<wire x1="210.82" y1="64.77" x2="212.09" y2="64.77" width="0.1524" layer="91"/>
-<wire x1="212.09" y1="64.77" x2="212.09" y2="63.5" width="0.1524" layer="91"/>
-<pinref part="C1" gate="G$1" pin="-"/>
-<wire x1="212.09" y1="63.5" x2="218.44" y2="63.5" width="0.1524" layer="91"/>
-<wire x1="218.44" y1="63.5" x2="226.06" y2="63.5" width="0.1524" layer="91"/>
-<junction x="218.44" y="63.5"/>
-<label x="228.6" y="63.5" size="1.778" layer="95"/>
+<pinref part="U$3" gate="G$1" pin="GND@0"/>
+<wire x1="212.09" y1="152.4" x2="213.36" y2="152.4" width="0.1524" layer="91"/>
+<wire x1="213.36" y1="152.4" x2="213.36" y2="151.13" width="0.1524" layer="91"/>
+<pinref part="C3" gate="G$1" pin="-"/>
+<wire x1="213.36" y1="151.13" x2="219.71" y2="151.13" width="0.1524" layer="91"/>
+<wire x1="219.71" y1="151.13" x2="227.33" y2="151.13" width="0.1524" layer="91"/>
+<junction x="219.71" y="151.13"/>
+<label x="229.87" y="151.13" size="1.778" layer="95"/>
 </segment>
 <segment>
@@
 </segment>
 <segment>
-<pinref part="U$3" gate="G$1" pin="GND@0"/>
-<wire x1="212.09" y1="152.4" x2="213.36" y2="152.4" width="0.1524" layer="91"/>
-<wire x1="213.36" y1="152.4" x2="213.36" y2="151.13" width="0.1524" layer="91"/>
-<pinref part="C3" gate="G$1" pin="-"/>
-<wire x1="213.36" y1="151.13" x2="219.71" y2="151.13" width="0.1524" layer="91"/>
-<wire x1="219.71" y1="151.13" x2="227.33" y2="151.13" width="0.1524" layer="91"/>
-<junction x="219.71" y="151.13"/>
-<label x="229.87" y="151.13" size="1.778" layer="95"/>
+<pinref part="U$4" gate="G$1" pin="GND@0"/>
+<wire x1="210.82" y1="64.77" x2="212.09" y2="64.77" width="0.1524" layer="91"/>
+<wire x1="212.09" y1="64.77" x2="212.09" y2="63.5" width="0.1524" layer="91"/>
+<pinref part="C1" gate="G$1" pin="-"/>
+<wire x1="212.09" y1="63.5" x2="218.44" y2="63.5" width="0.1524" layer="91"/>
+<wire x1="218.44" y1="63.5" x2="226.06" y2="63.5" width="0.1524" layer="91"/>
+<junction x="218.44" y="63.5"/>
+<label x="228.6" y="63.5" size="1.778" layer="95"/>
 </segment>
 <segment>

Commit message: primeira versao completa da board
Parts:
- added GOLD_ORB_SM1: OSHWLOGO_GOLD_ORB_SM, NBitWonder:OSHWLOGO_GOLD_ORB_SM
- C1, C2, C3: value (none) -> 10UF/30V
- X1: value (none) -> MOTOR 1
- X2: value (none) -> MOTOR 2
- X3: value (none) -> MOTOR 3
- renumbered S1 to FEED, S2 to START, S3 to RESET
Connections:
- removed net N$22: U$1.D8
- net ENABLE: now also U$1.D8
Other:
- note added: "OpenSourceHardware Logo"
Changed lines of the file:
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@@
 <setting verticaltext="up"/>
 </settings>
-<grid distance="0.05" unitdist="inch" unit="inch" style="lines" multiple="1" display="yes" altdistance="0.01" altunitdist="inch" altunit="inch"/>
+<grid distance="0.1" unitdist="inch" unit="inch" style="lines" multiple="1" display="no" altdistance="0.01" altunitdist="inch" altunit="inch"/>
 <layers>
 <layer number="1" name="Top" color="4" fill="1" visible="no" active="no"/>
@@
 <layer number="121" name="_tsilk" color="7" fill="1" visible="yes" active="yes"/>
 <layer number="122" name="_bsilk" color="7" fill="1" visible="yes" active="yes"/>
+<layer number="125" name="_tNames" color="7" fill="1" visible="yes" active="yes"/>
+<layer number="144" name="Drill_legend" color="7" fill="1" visible="yes" active="yes"/>
 <layer number="151" name="HeatSink" color="7" fill="1" visible="yes" active="yes"/>
 <layer number="200" name="200bmp" color="1" fill="10" visible="yes" active="yes"/>
@@
 <layer number="207" name="207bmp" color="8" fill="10" visible="yes" active="yes"/>
 <layer number="208" name="208bmp" color="9" fill="10" visible="yes" active="yes"/>
+<layer number="209" name="209bmp" color="7" fill="1" visible="yes" active="yes"/>
+<layer number="210" name="210bmp" color="7" fill="1" visible="yes" active="yes"/>
+<layer number="211" name="211bmp" color="7" fill="1" visible="yes" active="yes"/>
+<layer number="212" name="212bmp" color="7" fill="1" visible="yes" active="yes"/>
+<layer number="213" name="213bmp" color="7" fill="1" visible="yes" active="yes"/>
+<layer number="214" name="214bmp" color="7" fill="1" visible="yes" active="yes"/>
+<layer number="215" name="215bmp" color="7" fill="1" visible="yes" active="yes"/>
+<layer number="216" name="216bmp" color="7" fill="1" visible="yes" active="yes"/>
 <layer number="250" name="Descript" color="3" fill="1" visible="no" active="no"/>
 <layer number="251" name="SMDround" color="12" fill="11" visible="no" active="no"/>
@@
 <part name="U$1" library="Arduino-clone" deviceset="NANO" device=""/>
 <part name="U$4" library="RepRapjr" deviceset="A4988BREAKOUT" device=""/>
-<part name="C1" library="rcl" deviceset="CPOL-US" device="E2.5-6"/>
-<part name="X1" library="con-phoenix-254" deviceset="MPT4" device=""/>
+<part name="C1" library="rcl" deviceset="CPOL-US" device="E2.5-6" value="10UF/30V"/>
+<part name="X1" library="con-phoenix-254" deviceset="MPT4" device="" value="MOTOR 1"/>
 <part name="SUPPLY1" library="supply2" deviceset="VCC" device=""/>
 <part name="GND1" library="supply1" deviceset="GND" device=""/>
@@
 <part name="SUPPLY2" library="supply2" deviceset="VCC" device=""/>
 <part name="U$2" library="RepRapjr" deviceset="A4988BREAKOUT" device=""/>
-<part name="C2" library="rcl" deviceset="CPOL-US" device="E2.5-6"/>
-<part name="X2" library="con-phoenix-254" deviceset="MPT4" device=""/>
+<part name="C2" library="rcl" deviceset="CPOL-US" device="E2.5-6" value="10UF/30V"/>
+<part name="X2" library="con-phoenix-254" deviceset="MPT4" device="" value="MOTOR 2"/>
 <part name="SUPPLY3" library="supply2" deviceset="VCC" device=""/>
 <part name="GND2" library="supply1" deviceset="GND" device=""/>
@@
 <part name="SUPPLY4" library="supply2" deviceset="VCC" device=""/>
 <part name="U$3" library="RepRapjr" deviceset="A4988BREAKOUT" device=""/>
-<part name="C3" library="rcl" deviceset="CPOL-US" device="E2.5-6"/>
-<part name="X3" library="con-phoenix-254" deviceset="MPT4" device=""/>
+<part name="C3" library="rcl" deviceset="CPOL-US" device="E2.5-6" value="10UF/30V"/>
+<part name="X3" library="con-phoenix-254" deviceset="MPT4" device="" value="MOTOR 3"/>
 <part name="SUPPLY5" library="supply2" deviceset="VCC" device=""/>
 <part name="GND3" library="supply1" deviceset="GND" device=""/>
@@
 <part name="SUPPLY6" library="supply2" deviceset="VCC" device=""/>
 <part name="X4" library="con-phoenix-350" deviceset="1751248" device=""/>
-<part name="S1" library="RepRapjr" deviceset="10-XX-RPAD" device=""/>
-<part name="S2" library="RepRapjr" deviceset="10-XX-RPAD" device=""/>
-<part name="S3" library="RepRapjr" deviceset="10-XX-RPAD" device=""/>
+<part name="FEED" library="RepRapjr" deviceset="10-XX-RPAD" device=""/>
+<part name="START" library="RepRapjr" deviceset="10-XX-RPAD" device=""/>
+<part name="RESET" library="RepRapjr" deviceset="10-XX-RPAD" device=""/>
 <part name="GND4" library="supply1" deviceset="GND" device=""/>
 <part name="SUPPLY7" library="supply2" deviceset="VCC" device=""/>
 <part name="GND5" library="supply1" deviceset="GND" device=""/>
+<part name="GOLD_ORB_SM1" library="NBitWonder" deviceset="OSHWLOGO" device="_GOLD_ORB_SM"/>
 </parts>
 <sheets>
 <sheet>
 <plain>
+<text x="20.32" y="30.48" size="1.778" layer="91">OpenSourceHardware Logo</text>
 </plain>
 <instances>
@@
 <instance part="X4" gate="-1" x="97.79" y="148.59" rot="R180"/>
 <instance part="X4" gate="-2" x="97.79" y="156.21" rot="R180"/>
-<instance part="S1" gate="1" x="34.29" y="77.47" rot="R270"/>
-<instance part="S2" gate="1" x="34.29" y="66.04" rot="R270"/>
-<instance part="S3" gate="1" x="34.29" y="87.63" rot="R270"/>
+<instance part="FEED" gate="1" x="34.29" y="77.47" rot="R270"/>
+<instance part="START" gate="1" x="34.29" y="66.04" rot="R270"/>
+<instance part="RESET" gate="1" x="34.29" y="87.63" rot="R270"/>
 <instance part="GND4" gate="1" x="24.13" y="58.42"/>
 <instance part="SUPPLY7" gate="G$1" x="58.42" y="78.74"/>
 <instance part="GND5" gate="1" x="58.42" y="66.04"/>
+<instance part="GOLD_ORB_SM1" gate="G$1" x="20.32" y="17.78"/>
 </instances>
 <busses>
@@
 </segment>
 <segment>
-<pinref part="S3" gate="1" pin="P"/>
+<pinref part="RESET" gate="1" pin="P"/>
 <pinref part="GND4" gate="1" pin="GND"/>
 <wire x1="29.21" y1="87.63" x2="24.13" y2="87.63" width="0.1524" layer="91"/>
 <wire x1="24.13" y1="87.63" x2="24.13" y2="77.47" width="0.1524" layer="91"/>
-<pinref part="S1" gate="1" pin="P"/>
+<pinref part="FEED" gate="1" pin="P"/>
 <wire x1="24.13" y1="77.47" x2="24.13" y2="66.04" width="0.1524" layer="91"/>
 <wire x1="24.13" y1="66.04" x2="24.13" y2="60.96" width="0.1524" layer="91"/>
 <wire x1="29.21" y1="77.47" x2="24.13" y2="77.47" width="0.1524" layer="91"/>
 <junction x="24.13" y="77.47"/>
-<pinref part="S2" gate="1" pin="P"/>
+<pinref part="START" gate="1" pin="P"/>
 <wire x1="29.21" y1="66.04" x2="24.13" y2="66.04" width="0.1524" layer="91"/>
 <junction x="24.13" y="66.04"/>
@@
 <label x="151.13" y="154.94" size="1.778" layer="95"/>
 </segment>
+<segment>
+<pinref part="U$1" gate="G$1" pin="D8"/>
+<wire x1="96.52" y1="92.71" x2="102.87" y2="92.71" width="0.1524" layer="91"/>
+<label x="104.14" y="92.71" size="1.778" layer="95"/>
+</segment>
 </net>
 <net name="N$2" class="0">
@@
 </segment>
 </net>
-<net name="N$22" class="0">
-<segment>
-<pinref part="U$1" gate="G$1" pin="D8"/>
-<wire x1="96.52" y1="92.71" x2="102.87" y2="92.71" width="0.1524" layer="91"/>
-<label x="104.14" y="92.71" size="1.778" layer="95"/>
-</segment>
-</net>
 <net name="N$16" class="0">
 <segment>
@@
 <wire x1="63.5" y1="95.25" x2="43.18" y2="95.25" width="0.1524" layer="91"/>
 <wire x1="43.18" y1="95.25" x2="43.18" y2="87.63" width="0.1524" layer="91"/>
-<pinref part="S3" gate="1" pin="S"/>
+<pinref part="RESET" gate="1" pin="S"/>
 <wire x1="43.18" y1="87.63" x2="39.37" y2="87.63" width="0.1524" layer="91"/>
 </segment>
@@
 <net name="N$17" class="0">
 <segment>
-<pinref part="S1" gate="1" pin="S"/>
+<pinref part="FEED" gate="1" pin="S"/>
 <wire x1="39.37" y1="77.47" x2="45.72" y2="77.47" width="0.1524" layer="91"/>
 <wire x1="45.72" y1="77.47" x2="45.72" y2="92.71" width="0.1524" layer="91"/>
@@
 <net name="N$18" class="0">
 <segment>
-<pinref part="S2" gate="1" pin="S"/>
+<pinref part="START" gate="1" pin="S"/>
 <wire x1="39.37" y1="66.04" x2="48.26" y2="66.04" width="0.1524" layer="91"/>
 <wire x1="48.26" y1="66.04" x2="48.26" y2="90.17" width="0.1524" layer="91"/>
